File: Hardware/HardwareMV/Hardware.brd (EAGLE design)
At the start: 58.5 x 63.4 mm, 26 parts, among them IC1 74FST3257DR2G, J1 1x10 HEADER "A", J2 1x10 HEADER "B", J6 22-27-2051-05, Q1 200mA/40V, Q2 200mA/40V, U1 MAX3232, U2 L86-M33, U4 74HC4051D,652

Commit message: minor layout changes
Parts:
- R3, R4, R5, R6: device rcl:0207/7 -> rcl:0207/2V
- moved Q1 41.9 mm to (69.2, 47.9), turned to 180 degrees
- moved Q2 34.2 mm to (75.2, 47.9), turned to 180 degrees
- moved R3 33.8 mm to (67.7, 42.4), turned to 270 degrees
- moved R4 31.5 mm to (70.6, 42.4), turned to 90 degrees
- moved R5 29.0 mm to (73.8, 42.4), turned to 90 degrees
- moved R6 26.9 mm to (76.7, 42.4), turned to 270 degrees
- moved C11 9.67 mm to (72.5, 38.2), turned to 0 degrees
- moved J6 2.67 mm to (31.6, 2.92)
- moved U2 1.40 mm to (33.3, 32.1)
Routing:
- net +3V3: track 66.6 -> 52.7 mm
- net GND: track 215.2 -> 206.9 mm, vias 5 -> 6
- net N$52: track 0.00 -> 6.10 mm
- net N$55: track 0.00 -> 5.78 mm
- net N$54: track 0.00 -> 5.78 mm
- net N$57: track 0.00 -> 3.43 mm
- net N$23: track 34.5 -> 31.9 mm
- net N$20: track 28.4 -> 25.7 mm
- net N$24: track 21.2 -> 18.5 mm
- net N$22: track 28.0 -> 25.3 mm
- net N$10: track 35.3 -> 33.9 mm
- net N$8: track 22.8 -> 21.4 mm
