File: Hardware/Hardware/Hardware.brd (EAGLE design)
At the start: 58.4 x 63.4 mm, 12 parts, among them J1 1x10 HEADER "A", J2 1x10 HEADER "B", U1 MAX3232

Commit message: Merged and tidied up the circuit, did my part of PCB
Parts:
- added C11: 1uF, rcl:C025-024X044
- added IC1: 74FST3257DR2G, 74FST3257DR2G:SOIC127P600X175-16N
- added J6: 22-27-2051-05, con-molex:6410-05
- added Q1, Q2: 200mA/40V, SparkFun-DiscreteSemi:TO-92
- added R1, R2: (no value), rcl:0207/7
- added R3, R6: 1K, rcl:0207/7
- added R4, R5: 4.7K, rcl:0207/7
- added U2: L86-M33, L86-M33:SON254P1840X1840X40-12N
- added U4: 74HC4051D,652, 74HC4051D_652:SOIC127P600X175-16N
- U1: device SparkFun-IC-Comms:TSSOP16 -> SparkFun-IC-Comms:SO16
- moved J3 16.9 mm to (29.0, 46.9)
- moved C4 14.5 mm to (31.2, 18.7), turned to 0 degrees
- moved C1 13.9 mm to (34.9, 29.5)
- moved C2 13.6 mm to (34.9, 25.4)
- moved U1 13.6 mm to (29.2, 26.2)
- moved C5 9.98 mm to (23.6, 30.0), turned to 90 degrees
- moved C3 9.86 mm to (26.9, 18.7)
Connections:
- removed net N$9 (its old number): J1.4, U1.11
- new net +3V3: C5.2, IC1.16, J1.1, Q1.3, R3.2, U1.16, U2.10, U2.4, U2.5, U4.16
- new net N$10: IC1.5, U2.1
- new net N$11: IC1.3, U1.12
- new net N$17: IC1.6, U1.11
- new net N$18: IC1.1, J1.7
- new net N$19: IC1.15, J1.8
- new net N$20: J6.3, U4.13
- new net N$22: J6.2, U4.14
- new net N$23: J6.1, U4.15
- new net N$24: J6.4, U4.12
- new net N$25: R2.2, U4.3
- new net N$3: IC1.4, J1.3
- new net N$47: J1.2, R1.2, R2.1
- new net N$49: J2.8, U4.11
- new net N$50: J2.9, U4.10
- new net N$51: J2.10, U4.9
- new net N$52: C11.2, R4.1, R5.1
- new net N$53: C11.1, J2.2
- new net N$54: Q2.2, R5.2, R6.1
- new net N$55: Q1.2, R3.1, R4.2
- new net N$57: Q1.1, Q2.3
- net GND: now also IC1.8, J2.1, J6.5, Q2.1, R1.1, R6.2, U2.12, U2.3, U4.6, U4.7, U4.8
- net N$5: now also IC1.7, J1.4; no longer C5.2, J1.1, U1.16
- net N$8: now also IC1.2, U2.2; no longer J1.3, U1.12
Routing:
- net GND: track 0.00 -> 204.1 mm, vias 0 -> 4
- net +3V3: track 0.00 -> 66.6 mm, vias 0 -> 2
- net N$15: track 0.00 -> 48.3 mm
- net N$16: track 0.00 -> 39.1 mm
- net N$10: track 0.00 -> 35.3 mm, vias 0 -> 2
- net N$19: track 0.00 -> 26.1 mm
- net N$47: track 0.00 -> 25.1 mm, vias 0 -> 1
- net N$21: track 0.00 -> 24.3 mm, vias 0 -> 1
- net N$18: track 0.00 -> 24.2 mm
- net N$43: track 0.00 -> 24.1 mm, vias 0 -> 1
- net N$8: track 0.00 -> 22.8 mm
- net CUT: track 23.5 -> 45.9 mm
- net N$17: track 0.00 -> 21.7 mm, vias 0 -> 1
- net N$13: track 0.00 -> 21.7 mm
- net N$11: track 0.00 -> 20.6 mm, vias 0 -> 1
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Other:
- board size 58.4 x 63.4 mm -> 58.5 x 63.4 mm

Commit message: Changes in brd
Parts:
- added J4: 22-27-2021-02, con-molex:6410-02
- R3, R4, R5, R6: device rcl:0207/7 -> rcl:0207/2V
- moved Q1 42.9 mm to (48.9, 53.1), turned to 180 degrees
- moved Q2 35.0 mm to (54.9, 53.1), turned to 180 degrees
- moved R3 26.8 mm to (47.4, 47.6), turned to 270 degrees
- moved R4 25.7 mm to (50.3, 47.6), turned to 90 degrees
- moved R5 24.4 mm to (53.5, 47.6), turned to 90 degrees
- moved R6 24.3 mm to (56.4, 47.6), turned to 270 degrees
- moved C11 12.7 mm to (55.0, 43.7), turned to 0 degrees
- moved J6 2.67 mm to (31.6, 2.92)
- moved U2 1.40 mm to (33.3, 32.1)
- moved R2 1.30 mm to (45.5, 15.9)
Connections:
- net N$53: now also J4.1
- net N$57: now also J4.2
Routing:
- net N$47: track 25.1 -> 78.6 mm
- net N$23: track 0.00 -> 31.9 mm, vias 0 -> 1
- net N$53: track 0.00 -> 29.4 mm, vias 0 -> 1
- net N$20: track 0.00 -> 25.7 mm, vias 0 -> 1
- net +3V3: track 66.6 -> 92.0 mm, vias 2 -> 3
- net N$22: track 0.00 -> 25.3 mm, vias 0 -> 1
- net GND: track 204.1 -> 229.1 mm, vias 4 -> 7
- net N$24: track 0.00 -> 18.5 mm, vias 0 -> 1
- net N$57: track 0.00 -> 16.2 mm
- net N$25: track 0.00 -> 8.45 mm
- net N$52: track 0.00 -> 7.07 mm
- net N$49: track 0.00 -> 6.95 mm
- net N$51: track 0.00 -> 6.95 mm
- net N$50: track 0.00 -> 6.43 mm
- net N$55: track 0.00 -> 5.78 mm
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
Commit message: Added UART MUX support
Parts:
- removed C11: 1uF, rcl:C025-024X044
- removed J4: 22-27-2021-02, con-molex:6410-02
- removed Q1, Q2: 200mA/40V, SparkFun-DiscreteSemi:TO-92
- removed R3, R6: 1K, rcl:0207/2V
- removed R4, R5: 4.7K, rcl:0207/2V
- added U$4: KCVG084B16, KCVG084B16:KCVG084B16
Connections:
- removed net N$52: C11.2, R4.1, R5.1
- removed net N$53: C11.1, J2.2, J4.1
- removed net N$54: Q2.2, R5.2, R6.1
- removed net N$55: Q1.2, R3.1, R4.2
- removed net N$57: J4.2, Q1.1, Q2.3
- new net N$31: J2.2, U$4.P$1
- net +3V3: no longer Q1.3, R3.2
- net GND: now also U$4.P$2; no longer Q2.1, R6.2
Routing:
- net N$53: track 29.4 -> 0.00 mm, vias 1 -> 0
- net +3V3: track 92.0 -> 72.6 mm, vias 3 -> 2
- net GND: track 229.1 -> 212.5 mm, vias 7 -> 9
- net N$57: track 16.2 -> 0.00 mm
- net N$31: track 0.00 -> 14.3 mm
- net N$52: track 7.07 -> 0.00 mm
- net N$55: track 5.78 -> 0.00 mm
- net N$54: track 5.78 -> 0.00 mm
- net N$30: track 0.00 -> 3.05 mm
- net N$29: track 0.00 -> 3.05 mm
- net N$28: track 0.00 -> 3.05 mm
- net N$27: track 0.00 -> 2.75 mm
- net N$11: track 20.6 -> 22.6 mm
- added copper zone on layer 1, net GND
- added copper zone on layer 16, net GND
Other:
- board text added: "BOT"
- board text added: "D:/Users/Marius/Documents/Strathclyde/EE318/University_of_Strathclyde_Coat_of_Arms.bmp"
- board text added: "Drone Recovery System"
- board text added: "TOP"
